File: KiCad/LoRa_Hat.kicad_sch (KiCad schematic)
At the start: 27 parts, among them J1 GPIO, J2 OLED Display, J3 Ext, J4 Ext, J5 LoRa RF SMA, J6 PJ-036DH, J7 Conn_01x01_Female, J8 Conn_01x01_Female, SW1 SW_Push, SW2 SW_Push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

Commit message: Schema corrections for J1 and J2 to reflect PCB silk layer print
Connections:
- net +3V3: now also JP1.3 (B), JP2.1 (A); no longer JP1.1 (A), JP2.3 (B)
- net GND: now also JP1.1 (A), JP2.3 (B); no longer JP1.3 (B), JP2.1 (A)
Changed lines of the file:
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@@
   (title_block
     (title "LoRa Raspberry Pi HAT")
-    (date "2023-10-28")
-    (rev "1,1")
+    (date "2024-09-19")
+    (rev "1.2")
     (company "SWISS-ARTG")
   )
@@
     )
   )
-  (symbol (lib_id "Jumper:Jumper_3_Open") (at 251.46 46.99 90) (mirror x) (unit 1)
-    (in_bom yes) (on_board yes) (dnp no) (fields_autoplaced)
-    (property "Reference" "JP1" (at 249.8339 47.4238 90)
+  (symbol (lib_id "Jumper:Jumper_3_Open") (at 251.46 46.99 90) (unit 1)
+    (in_bom yes) (on_board yes) (dnp no)
+    (property "Reference" "JP1" (at 249.3258 47.3068 90)
       (effects (font (size 1.27 1.27)) (justify left))
     )
-    (property "Value" "Jumper_3_Bridged12" (at 249.8339 48.6922 90)
+    (property "Value" "Jumper_3_Bridged12" (at 249.8339 45.2878 90)
       (effects (font (size 1.27 1.27)) (justify left) hide)
     )
@@
     )
   )
-  (symbol (lib_id "Jumper:Jumper_3_Open") (at 264.16 46.99 90) (unit 1)
-    (in_bom yes) (on_board yes) (dnp no) (fields_autoplaced)
-    (property "Reference" "JP2" (at 262.5339 47.4238 90)
+  (symbol (lib_id "Jumper:Jumper_3_Open") (at 264.16 46.99 90) (mirror x) (unit 1)
+    (in_bom yes) (on_board yes) (dnp no)
+    (property "Reference" "JP2" (at 262.0258 47.3068 90)
       (effects (font (size 1.27 1.27)) (justify left))
     )
-    (property "Value" "Jumper_3_Bridged12" (at 262.5339 48.6922 90)
+    (property "Value" "Jumper_3_Bridged12" (at 262.5339 45.2878 90)
       (effects (font (size 1.27 1.27)) (justify left) hide)
     )
